Commit message: create arm

File: simbot_description/urdf/manipulator.urdf.xacro (robot description, xacro)
@@ -2,57 +2,87 @@
 <robot xmlns:xacro="https://www.ros.org/wiki/xacro">
     <xacro:property name="M_PI" value="3.1415926535897931" />
-    <xacro:property name="shoulder_mass" value="2"/>
-    <xacro:property name="shoulder_r" value="0.1"/>
-    <xacro:property name="shoulder_l" value="0.1"/>
-    <xacro:property name="upper_arm_mass" value="0.4"/>
-    <xacro:property name="upper_arm_r" value="0.05"/>
+    <xacro:property name="shoulder_0_mass" value="2"/>
+    <xacro:property name="shoulder_0_r" value="0.1"/>
+    <xacro:property name="shoulder_0_l" value="0.1"/>
+    <xacro:property name="shoulder_1_mass" value="0.4"/>
+    <xacro:property name="shoulder_1_r" value="0.05"/>
+    <xacro:property name="shoulder_1_l" value="0.12"/>
+    <xacro:property name="upper_arm_mass" value="0.2"/>
+    <xacro:property name="upper_arm_r" value="0.04"/>
     <xacro:property name="upper_arm_l" value="0.4"/>
-    <xacro:property name="elbow_mass" value="0.4"/>
-    <xacro:property name="elbow_r" value="0.05"/>
-    <xacro:property name="elbow_l" value="0.2"/>
-    <xacro:property name="lower_arm_mass" value="0.2"/>
-    <xacro:property name="lower_arm_r" value="0.04"/>
-    <xacro:property name="lower_arm_l" value="0.2"/>
+    <xacro:property name="elbow_mass" value="0.2"/>
+    <xacro:property name="elbow_r" value="0.02"/>
+    <xacro:property name="elbow_l" value="0.1"/>
+    <xacro:property name="lower_arm_mass" value="0.1"/>
+    <xacro:property name="lower_arm_r" value="0.02"/>
+    <xacro:property name="lower_arm_l" value="0.3"/>
     <xacro:property name="wrist_mass" value="0.1"/>
-    <xacro:property name="wrist_r" value="0.02"/>
+    <xacro:property name="wrist_r" value="0.05"/>
     <xacro:property name="wrist_l" value="0.02"/>
     <xacro:macro name="manipulator" params="parent name:=manipulator *origin">
-        <joint name="${parent}-${name}_shoulder" type="revolute">
+        <joint name="${parent}-${name}_shoulder_0" type="revolute">
             <xacro:insert_block name="origin" />
             <parent link="${parent}"/>
-            <child link="${name}_shoulder"/>
+            <child link="${name}_shoulder_0"/>
             <limit lower="${-19*M_PI/20}" upper="${19*M_PI/20}" effort="50" velocity="${M_PI}"/>
             <axis xyz="0 0 1"/>
         </joint>
-        <link name="${name}_shoulder">
-            <visual>
-                <origin rpy="0 0 0" xyz="0 0 0"/>
-                <geometry>
-                    <cylinder length="${shoulder_l}" radius="${shoulder_r}"/>
-                </geometry>
-                <material name="orange"/>
-            </visual>
-            <collision>
-                <origin rpy="0 0 0" xyz="0 0 0" />
-                <geometry>
-                    <cylinder length="${shoulder_l}" radius="${shoulder_r}"/>
-                </geometry>
-            </collision>
-            <inertial>
-				<mass value="${shoulder_mass}" />
-				<origin xyz="0 0 0" />
-				<inertia ixx="${1/12*shoulder_mass*(3*shoulder_r*shoulder_r+shoulder_l*shoulder_l)}" ixy="0" ixz="0" iyy="${1/12*shoulder_mass*(3*shoulder_r*shoulder_r+shoulder_l*shoulder_l)}" iyz="0" izz="${1/2*shoulder_mass*shoulder_r*shoulder_r}"/>
-			</inertial>
-		</link>
-        <joint name="${name}_shoulder-${name}_upper_arm" type="revolute">
-            <origin rpy="0 0 0" xyz="0 0 ${shoulder_l/2}"/>
-            <parent link="${name}_shoulder"/>
+        <link name="${name}_shoulder_0">
+            <visual>
+                <origin rpy="0 0 0" xyz="0 0 0"/>
+                <geometry>
+                    <cylinder length="${shoulder_0_l}" radius="${shoulder_0_r}"/>
+                </geometry>
+                <material name="orange"/>
+            </visual>
+            <collision>
+                <origin rpy="0 0 0" xyz="0 0 0" />
+                <geometry>
+                    <cylinder length="${shoulder_0_l}" radius="${shoulder_0_r}"/>
+                </geometry>
+            </collision>
+            <inertial>
+				<mass value="${shoulder_0_mass}" />
+				<origin xyz="0 0 0" />
+				<inertia ixx="${1/12*shoulder_0_mass*(3*shoulder_0_r*shoulder_0_r+shoulder_0_l*shoulder_0_l)}" ixy="0" ixz="0" iyy="${1/12*shoulder_0_mass*(3*shoulder_0_r*shoulder_0_r+shoulder_0_l*shoulder_0_l)}" iyz="0" izz="${1/2*shoulder_0_mass*shoulder_0_r*shoulder_0_r}"/>
+			</inertial>
+		</link>
+        <joint name="${name}_shoulder_0-${name}_shoulder_1" type="revolute">
+            <origin rpy="${-M_PI/2} 0 0" xyz="0 0 ${shoulder_0_l/2}"/>
+            <parent link="${name}_shoulder_0"/>
+            <child link="${name}_shoulder_1"/>
+            <limit lower="${-7*M_PI/12}" upper="${M_PI/12}" effort="50" velocity="${M_PI}"/>
+            <axis xyz="0 0 1"/>
+        </joint>
+        <link name="${name}_shoulder_1">
+            <visual>
+                <origin rpy="0 0 0" xyz="0 0 0"/>
+                <geometry>
+                    <cylinder length="${shoulder_1_l}" radius="${shoulder_1_r}"/>
+                </geometry>
+                <material name="orange"/>
+            </visual>
+            <collision>
+                <origin rpy="0 0 0" xyz="0 0 0" />
+                <geometry>
+                    <cylinder length="${shoulder_1_l}" radius="${shoulder_1_r}"/>
+                </geometry>
+            </collision>
+            <inertial>
+				<mass value="${shoulder_1_mass}" />
+				<origin xyz="0 0 0" />
+				<inertia ixx="${1/12*shoulder_1_mass*(3*shoulder_1_r*shoulder_1_r+shoulder_1_l*shoulder_1_l)}" ixy="0" ixz="0" iyy="${1/12*shoulder_1_mass*(3*shoulder_1_r*shoulder_1_r+shoulder_1_l*shoulder_1_l)}" iyz="0" izz="${1/2*shoulder_1_mass*shoulder_1_r*shoulder_1_r}"/>
+			</inertial>
+		</link>
+        <joint name="${name}_shoulder_1-${name}_upper_arm" type="revolute">
+            <origin rpy="0 ${-M_PI/2} 0" xyz="${upper_arm_l/2} 0 0"/>
+            <parent link="${name}_shoulder_1"/>
             <child link="${name}_upper_arm"/>
-            <limit lower="${-M_PI/6}" upper="${7*M_PI/12}" effort="50" velocity="${M_PI}"/>
-            <axis xyz="0 1 0"/>
+            <limit lower="0" upper="0" effort="0" velocity="0"/>
+            <axis xyz="1 0 0"/>
         </joint>
         <link name="${name}_upper_arm">
             <visual>
-                <origin rpy="0 0 0" xyz="0 0 ${upper_arm_l/2}"/>
+                <origin rpy="0 0 0" xyz="0 0 0"/>
                 <geometry>
                     <cylinder length="${upper_arm_l}" radius="${upper_arm_r}"/>
@@ -61,5 +91,5 @@
             </visual>
             <collision>
-                <origin rpy="0 0 0" xyz="0 0 ${upper_arm_l/2}" />
+                <origin rpy="0 0 0" xyz="0 0 0" />
                 <geometry>
                     <cylinder length="${upper_arm_l}" radius="${upper_arm_r}"/>
@@ -70,4 +100,85 @@
 				<origin xyz="0 0 0" />
 				<inertia ixx="${1/12*upper_arm_mass*(3*upper_arm_r*upper_arm_r+upper_arm_l*upper_arm_l)}" ixy="0" ixz="0" iyy="${1/12*upper_arm_mass*(3*upper_arm_r*upper_arm_r+upper_arm_l*upper_arm_l)}" iyz="0" izz="${1/2*upper_arm_mass*upper_arm_r*upper_arm_r}"/>
+			</inertial>
+		</link>
+        <joint name="${name}_upper_arm-${name}_elbow" type="revolute">
+            <origin rpy="0 ${-M_PI/2} 0" xyz="0 0 ${-upper_arm_l/2} "/>
+            <parent link="${name}_upper_arm"/>
+            <child link="${name}_elbow"/>
+            <limit lower="${-3*M_PI/5}" upper="${3*M_PI/5}" effort="50" velocity="${M_PI}"/>
+            <axis xyz="0 0 1"/>
+        </joint>
+        <link name="${name}_elbow">
+            <visual>
+                <origin rpy="0 0 0" xyz="0 0 0"/>
+                <geometry>
+                    <cylinder length="${elbow_l}" radius="${elbow_r}"/>
+                </geometry>
+                <material name="orange"/>
+            </visual>
+            <collision>
+                <origin rpy="0 0 0" xyz="0 0 0" />
+                <geometry>
+                    <cylinder length="${elbow_l}" radius="${elbow_r}"/>
+                </geometry>
+            </collision>
+            <inertial>
+				<mass value="${elbow_mass}" />
+				<origin xyz="0 0 0" />
+				<inertia ixx="${1/12*elbow_mass*(3*elbow_r*elbow_r+elbow_l*elbow_l)}" ixy="0" ixz="0" iyy="${1/12*elbow_mass*(3*elbow_r*elbow_r+elbow_l*elbow_l)}" iyz="0" izz="${1/2*elbow_mass*elbow_r*elbow_r}"/>
+			</inertial>
+		</link>
+        <joint name="${name}_elbow-${name}_lower_arm" type="revolute">
+            <origin rpy="0 ${-M_PI/2} 0" xyz="${-lower_arm_l/2} 0 0"/>
+            <parent link="${name}_elbow"/>
+            <child link="${name}_lower_arm"/>
+            <limit lower="0" upper="0" effort="0" velocity="0"/>
+            <axis xyz="0 0 1"/>
+        </joint>
+        <link name="${name}_lower_arm">
+            <visual>
+                <origin rpy="0 0 0" xyz="0 0 0"/>
+                <geometry>
+                    <cylinder length="${lower_arm_l}" radius="${lower_arm_r}"/>
+                </geometry>
+                <material name="orange"/>
+            </visual>
+            <collision>
+                <origin rpy="0 0 0" xyz="0 0 0" />
+                <geometry>
+                    <cylinder length="${lower_arm_l}" radius="${lower_arm_r}"/>
+                </geometry>
+            </collision>
+            <inertial>
+				<mass value="${lower_arm_mass}" />
+				<origin xyz="0 0 0" />
+				<inertia ixx="${1/12*lower_arm_mass*(3*lower_arm_r*lower_arm_r+lower_arm_l*lower_arm_l)}" ixy="0" ixz="0" iyy="${1/12*lower_arm_mass*(3*lower_arm_r*lower_arm_r+lower_arm_l*lower_arm_l)}" iyz="0" izz="${1/2*lower_arm_mass*lower_arm_r*lower_arm_r}"/>
+			</inertial>
+		</link>
+        <joint name="${name}_lower_arm-${name}_wrist" type="revolute">
+            <origin rpy="0 0 0" xyz="0 0 ${lower_arm_l/2+wrist_l/2}"/>
+            <parent link="${name}_lower_arm"/>
+            <child link="${name}_wrist"/>
+            <limit lower="${-19*M_PI/20}" upper="${19*M_PI/20}" effort="50" velocity="${M_PI}"/>
+            <axis xyz="0 0 1"/>
+        </joint>
+        <link name="${name}_wrist">
+            <visual>
+                <origin rpy="0 0 0" xyz="0 0 0"/>
+                <geometry>
+                    <cylinder length="${wrist_l}" radius="${wrist_r}"/>
+                </geometry>
+                <material name="orange"/>
+            </visual>
+            <collision>
+                <origin rpy="0 0 0" xyz="0 0 0" />
+                <geometry>
+                    <cylinder length="${wrist_l}" radius="${wrist_r}"/>
+                </geometry>
+            </collision>
+            <inertial>
+				<mass value="${wrist_mass}" />
+				<origin xyz="0 0 0" />
+				<inertia ixx="${1/12*wrist_mass*(3*wrist_r*wrist_r+wrist_l*wrist_l)}" ixy="0" ixz="0" iyy="${1/12*wrist_mass*(3*wrist_r*wrist_r+wrist_l*wrist_l)}" iyz="0" izz="${1/2*wrist_mass*wrist_r*wrist_r}"/>
 			</inertial>
 		</link>

File: simbot_description/urdf/triwheeler_manipulator_rgbd.urdf.xacro (robot description, xacro)
@@ -12,5 +12,5 @@
     <xacro:include filename="$(find simbot_description)/urdf/manipulator.urdf.xacro" />
     <xacro:manipulator parent="chassis">
-        <origin xyz="${2*chassis_x/5} 0.0 ${chassis_z/2+shoulder_l/2}" rpy="0 0 0"/>
+        <origin xyz="${2*chassis_x/5} 0.0 ${chassis_z/2+shoulder_0_l/2}" rpy="0 0 0"/>
     </xacro:manipulator>
 </robot>

Commit message: add gripper

File: simbot_description/urdf/manipulator.urdf.xacro (robot description, xacro)
@@ -9,5 +9,5 @@
     <xacro:property name="shoulder_1_l" value="0.12"/>
     <xacro:property name="upper_arm_mass" value="0.2"/>
-    <xacro:property name="upper_arm_r" value="0.04"/>
+    <xacro:property name="upper_arm_r" value="0.03"/>
     <xacro:property name="upper_arm_l" value="0.4"/>
     <xacro:property name="elbow_mass" value="0.2"/>
@@ -20,4 +20,12 @@
     <xacro:property name="wrist_r" value="0.05"/>
     <xacro:property name="wrist_l" value="0.02"/>
+    <xacro:property name="gripper_mass" value="0.2"/>
+    <xacro:property name="gripper_x" value="0.14"/>
+    <xacro:property name="gripper_y" value="0.07"/>
+    <xacro:property name="gripper_z" value="0.04"/>
+    <xacro:property name="finger_mass" value="0.02"/>
+    <xacro:property name="finger_x" value="0.02"/>
+    <xacro:property name="finger_y" value="0.07"/>
+    <xacro:property name="finger_z" value="0.07"/>
     <xacro:macro name="manipulator" params="parent name:=manipulator *origin">
         <joint name="${parent}-${name}_shoulder_0" type="revolute">
@@ -88,5 +96,5 @@
                     <cylinder length="${upper_arm_l}" radius="${upper_arm_r}"/>
                 </geometry>
-                <material name="orange"/>
+                <material name="grey"/>
             </visual>
             <collision>
@@ -142,5 +150,5 @@
                     <cylinder length="${lower_arm_l}" radius="${lower_arm_r}"/>
                 </geometry>
-                <material name="orange"/>
+                <material name="grey"/>
             </visual>
             <collision>
@@ -183,71 +191,85 @@
 			</inertial>
 		</link>
-        <!-- <joint name="camera_holder-camera_body" type="revolute">
-            <origin rpy="0 0 0" xyz="0 0 ${holder_l/2+camera_height/2}"/>
-            <parent link="camera_holder"/>
-            <child link="camera_body"/>
-            <limit lower="${-M_PI/6}" upper="${M_PI/12}" effort="50" velocity="${M_PI}"/>
-            <axis xyz="0 1 0"/>
-        </joint>
-        <link name="camera_body">
-			<visual>
-				<origin xyz="0 0 0" rpy="0 0 0" />
-				<geometry>
-					<box size="${camera_depth} ${camera_width} ${camera_height}" />
-				</geometry>
-                <color rgba="0.5 0.5 0.5 1"/>
-			</visual>
-			<collision>
-				<origin xyz="0 0 0" rpy="0 0 0" />
-				<geometry>
-                    <box size="${camera_depth} ${camera_width} ${camera_height}" />
-				</geometry>
-			</collision>
-            <inertial>
-				<mass value="${camera_mass}" />
-				<origin xyz="0 0 0" />
-				<inertia ixx="5.8083e-4" ixy="0" ixz="0" iyy="3.0833e-5" iyz="0" izz="5.9083e-4" />
-			</inertial>
-		</link>
-        <joint name="camera_body-depth_frame" type="fixed">
-            <origin xyz="${camera_depth/2} 0.0175 0.0" rpy="${-M_PI/2} 0 ${-M_PI/2}" />
-            <parent link="camera_body" />
-            <child link="camera_depth_frame"/>
-        </joint>
-        <link name="camera_depth_frame"/>
-        <joint name="camera_body-depth_optical" type="fixed">
-            <origin xyz="${camera_depth/2} 0.0175 0" rpy="0 0 0" />
-            <parent link="camera_body" />
-            <child link="camera_depth_optical"/>
-        </joint>
-        <link name="camera_depth_optical"/>
-    </xacro:macro>
-    <xacro:macro name="rgbd_camera_gazebo_plugin_macro" params="link_name camera_name:=camera frame_name">
-        <gazebo reference="${link_name}">
-            <sensor type="depth" name="${link_name}_camera">
-                <update_rate>30</update_rate>
-                <camera>
-                    <horizontal_fov>${69.4 * M_PI/180.0}</horizontal_fov>
-                    <image>
-                        <format>B8G8R8</format>
-                        <width>640</width>
-                        <height>480</height>
-                    </image>
-                    <clip>
-                        <near>0.3</near>
-                        <far>10</far>
-                    </clip>
-                </camera>
-                <plugin name="${link_name}_controller" filename="libgazebo_ros_openni_kinect.so">
-                    <cameraName>${camera_name}</cameraName>
-                    <imageTopicName>/${camera_name}/color/image_raw</imageTopicName>
-                    <cameraInfoTopicName>/${camera_name}/color/camera_info</cameraInfoTopicName>
-                    <depthImageTopicName>/${camera_name}/depth/image_raw</depthImageTopicName>
-                    <depthImageInfoTopicName>/${camera_name}/depth/camera_info</depthImageInfoTopicName>
-                    <pointCloudTopicName>/${camera_name}/depth/points</pointCloudTopicName>
-                    <frameName>${frame_name}</frameName>
-                </plugin>
-            </sensor>
-        </gazebo> -->
+        <joint name="${name}_wrist-${name}_gripper" type="revolute">
+            <origin rpy="0 0 0" xyz="0 0 ${wrist_l/2+gripper_z/2}"/>
+            <parent link="${name}_wrist"/>
+            <child link="${name}_gripper"/>
+            <limit lower="0" upper="0" effort="0" velocity="0"/>
+            <axis xyz="0 0 1"/>
+        </joint>
+        <link name="${name}_gripper">
+            <visual>
+                <origin xyz="0 0 0" rpy="0 0 0" />
+                <geometry>
+                    <box size="${gripper_x} ${gripper_y} ${gripper_z}"/> />
+                </geometry>
+                <material name="grey"/>
+            </visual>
+            <collision>
+                <origin xyz="0 0 0" rpy="0 0 0" />
+                <geometry>
+                    <box size="${gripper_x} ${gripper_y} ${gripper_z}"/> />
+                </geometry>
+            </collision>
+            <inertial>
+				<mass value="${gripper_mass}" />
+				<origin xyz="0 0 0" />
+                <inertia ixx="${1/12*gripper_mass*(gripper_y*gripper_y+gripper_z*gripper_z)}" ixy="0" ixz="0" iyy="${1/12*gripper_mass*(gripper_z*gripper_z+gripper_x*gripper_x)}" iyz="0" izz="${1/12*gripper_mass*(gripper_x*gripper_x+gripper_y*gripper_y)}"/>
+            </inertial>
+		</link>
+        <joint name="${name}_gripper-${name}_left_finger" type="prismatic">
+            <origin rpy="0 0 0" xyz="${-gripper_x/2+finger_x/2} 0 ${gripper_z/2+finger_z/2}"/>
+            <parent link="${name}_gripper"/>
+            <child link="${name}_left_finger"/>
+            <limit lower="0" upper="${gripper_x/2-finger_x}" effort="70" velocity="2"/>
+            <axis xyz="1 0 0"/>
+        </joint>
+        <link name="${name}_left_finger">
+            <visual>
+                <origin xyz="0 0 0" rpy="0 0 0" />
+                <geometry>
+                    <box size="${finger_x} ${finger_y} ${finger_z}"/> />
+                </geometry>
+                <material name="white"/>
+            </visual>
+            <collision>
+                <origin xyz="0 0 0" rpy="0 0 0" />
+                <geometry>
+                    <box size="${finger_x} ${finger_y} ${finger_z}"/> />
+                </geometry>
+            </collision>
+            <inertial>
+				<mass value="${finger_mass}" />
+				<origin xyz="0 0 0" />
+                <inertia ixx="${1/12*finger_mass*(finger_y*finger_y+finger_z*finger_z)}" ixy="0" ixz="0" iyy="${1/12*finger_mass*(finger_z*finger_z+finger_x*finger_x)}" iyz="0" izz="${1/12*finger_mass*(finger_x*finger_x+finger_y*finger_y)}"/>
+            </inertial>
+		</link>
+        <joint name="${name}_gripper-${name}_right_finger" type="prismatic">
+            <origin rpy="0 0 0" xyz="${gripper_x/2-finger_x/2} 0 ${gripper_z/2+finger_z/2}"/>
+            <parent link="${name}_gripper"/>
+            <child link="${name}_right_finger"/>
+            <limit lower="${-gripper_x/2+finger_x}" upper="0" effort="70" velocity="2"/>
+            <axis xyz="1 0 0"/>
+        </joint>
+        <link name="${name}_right_finger">
+            <visual>
+                <origin xyz="0 0 0" rpy="0 0 0" />
+                <geometry>
+                    <box size="${finger_x} ${finger_y} ${finger_z}"/> />
+                </geometry>
+                <material name="white"/>
+            </visual>
+            <collision>
+                <origin xyz="0 0 0" rpy="0 0 0" />
+                <geometry>
+                    <box size="${finger_x} ${finger_y} ${finger_z}"/> />
+                </geometry>
+            </collision>
+            <inertial>
+				<mass value="${finger_mass}" />
+				<origin xyz="0 0 0" />
+                <inertia ixx="${1/12*finger_mass*(finger_y*finger_y+finger_z*finger_z)}" ixy="0" ixz="0" iyy="${1/12*finger_mass*(finger_z*finger_z+finger_x*finger_x)}" iyz="0" izz="${1/12*finger_mass*(finger_x*finger_x+finger_y*finger_y)}"/>
+            </inertial>
+		</link>
     </xacro:macro>
 </robot>

File: simbot_description/urdf/triwheeler_base.urdf.xacro (robot description, xacro)
@@ -7,5 +7,5 @@
     <xacro:property name="chassis_y" value="0.6" />
     <xacro:property name="chassis_z" value="0.2" />
-    <xacro:property name="chassis_m" value="1" />
+    <xacro:property name="chassis_m" value="4" />
     <!-- properties of plate link -->
     <xacro:property name="plate_r" value="0.35"/>
@@ -15,5 +15,5 @@
     <xacro:property name="support_r" value="0.2"/>
     <xacro:property name="support_l" value="0.15"/>
-    <xacro:property name="support_m" value="0.4"/>
+    <xacro:property name="support_m" value="0.8"/>
     <!-- properties of link_caster -->
     <xacro:property name="caster_r" value="0.1"/>
