Commit message: create laser range sensor

File: simbot_description/urdf/rgbd_camera.urdf.xacro (robot description, xacro)
@@ -32,7 +32,7 @@
             </collision>
             <inertial>
-				<mass value="${camera_mass}" />
+				<mass value="${holder_mass}" />
 				<origin xyz="0 0 0" />
-				<inertia ixx="${1/12*camera_mass*(3*holder_r*holder_r+holder_l*holder_l)}" ixy="0" ixz="0" iyy="${1/12*holder_mass*(3*holder_r*holder_r+holder_l*holder_l)}" iyz="0" izz="${1/2*holder_mass*holder_r*holder_r}"/>
+				<inertia ixx="${1/12*holder_mass*(3*holder_r*holder_r+holder_l*holder_l)}" ixy="0" ixz="0" iyy="${1/12*holder_mass*(3*holder_r*holder_r+holder_l*holder_l)}" iyz="0" izz="${1/2*holder_mass*holder_r*holder_r}"/>
 			</inertial>
 		</link>

Commit message: create imu

File: simbot_description/urdf/rgbd_camera.urdf.xacro (robot description, xacro)
@@ -76,6 +76,32 @@
         </joint>
         <link name="camera_depth_optical"/>
+        <gazebo reference="camera_depth_optical">
+            <sensor type="depth" name="camera">
+                <update_rate>30</update_rate>
+                <camera>
+                    <horizontal_fov>${69.4 * M_PI/180.0}</horizontal_fov>
+                    <image>
+                        <format>B8G8R8</format>
+                        <width>640</width>
+                        <height>480</height>
+                    </image>
+                    <clip>
+                        <near>0.3</near>
+                        <far>10</far>
+                    </clip>
+                </camera>
+                <plugin name="camera_controller" filename="libgazebo_ros_openni_kinect.so">
+                    <cameraName>camera</cameraName>
+                    <imageTopicName>/camera/color/image_raw</imageTopicName>
+                    <cameraInfoTopicName>/camera/color/camera_info</cameraInfoTopicName>
+                    <depthImageTopicName>/camera/depth/image_raw</depthImageTopicName>
+                    <depthImageInfoTopicName>/camera/depth/camera_info</depthImageInfoTopicName>
+                    <pointCloudTopicName>/camera/depth/points</pointCloudTopicName>
+                    <frameName>camera</frameName>
+                </plugin>
+            </sensor>
+        </gazebo>
     </xacro:macro>
-    <xacro:macro name="rgbd_camera_gazebo_plugin_macro" params="link_name camera_name:=camera frame_name">
+    <!-- <xacro:macro name="rgbd_camera_gazebo_plugin_macro" params="link_name camera_name:=camera frame_name">
         <gazebo reference="${link_name}">
             <sensor type="depth" name="${link_name}_camera">
@@ -104,4 +130,4 @@
             </sensor>
         </gazebo>
-    </xacro:macro>
+    </xacro:macro> -->
 </robot>

File: simbot_description/urdf/triwheeler_base.urdf.xacro (robot description, xacro)
@@ -193,4 +193,12 @@
             </inertial>
         </link>
+        <joint name="chassis-imu" type="revolute">
+            <origin rpy="0 0 0" xyz="${chassis_x/4} 0 ${chassis_z/2}"/>
+            <parent link="chassis"/>
+            <child link="imu"/>
+            <limit lower="0" upper="0" effort="0" velocity="0"/>
+            <axis xyz="0 0 1"/>
+        </joint>
+        <link name="imu"/>
         <transmission name="left_wheel-trans" type="simpletransmission">
             <type>transmission_interface/simpletransmission</type>
@@ -211,4 +219,23 @@
             </joint>
         </transmission>
+        <gazebo reference="imu">
+            <gravity>true</gravity>
+            <sensor name="imu_sensor" type="imu">
+                <always_on>true</always_on>
+                <update_rate>100</update_rate>
+                <visualize>true</visualize>
+                <topic>__default_topic__</topic>
+                <plugin filename="libgazebo_ros_imu_sensor.so" name="imu_plugin">
+                    <topicName>imu</topicName>
+                    <bodyName>imu_link</bodyName>
+                    <updateRateHZ>10.0</updateRateHZ>
+                    <gaussianNoise>0.0</gaussianNoise>
+                    <xyzOffset>0 0 0</xyzOffset>
+                    <rpyOffset>0 0 0</rpyOffset>
+                    <frameName>imu_link</frameName>
+                </plugin>
+                <pose>0 0 0 0 0 0</pose>
+            </sensor>
+        </gazebo>
     </xacro:macro>
 </robot>
