Commit message: swap "triwheeler" and "triwheeler_base"

File: simbot_description/urdf/triwheeler_base.urdf.xacro (robot description, xacro)
@@ -1,241 +1,7 @@
-<?xml version="1.0" ?>
-<robot xmlns:xacro="https://www.ros.org/wiki/xacro" >
-    <!-- constants for robot dimensions -->
-    <xacro:property name="PI" value="3.1415926535897931"/>
-    <!-- properties of chassis link -->
-    <xacro:property name="chassis_x" value="0.8" />
-    <xacro:property name="chassis_y" value="0.6" />
-    <xacro:property name="chassis_z" value="0.2" />
-    <xacro:property name="chassis_m" value="4" />
-    <!-- properties of plate link -->
-    <xacro:property name="plate_r" value="0.35"/>
-    <xacro:property name="plate_l" value="0.04"/>
-    <xacro:property name="plate_m" value="0.2"/>
-    <!-- properties of plate support link -->
-    <xacro:property name="support_r" value="0.2"/>
-    <xacro:property name="support_l" value="0.15"/>
-    <xacro:property name="support_m" value="0.8"/>
-    <!-- properties of link_caster -->
-    <xacro:property name="caster_r" value="0.1"/>
-    <xacro:property name="caster_m" value="0.1"/>
-    <!-- properties of wheel -->
-    <xacro:property name="wheel_r" value="0.2"/>
-    <xacro:property name="wheel_l" value="0.08"/>
-    <xacro:property name="wheel_m" value="0.5"/>
-    <!-- wheel mounting positions -->
-    <xacro:property name="wheelbase" value="0.7" />
-    <xacro:property name="track" value="0.7" />
-    <!-- import all gazebo-customization elements, including gazebo colors -->
-    <!-- <xacro:include filename="$(find simbot_description)/urdf/tri_wheeler.gazebo" /> -->
-    <!-- import rviz colors -->
-    <xacro:include filename="$(find simbot_description)/urdf/materials.urdf.xacro" />
-    <!-- main triwheeler link -->
-    <xacro:macro name="triwheeler_base_macro">
-        <!-- chassis is the center of the robot's bottom plate -->
-        <link name="chassis">
-            <visual>
-                <origin xyz="0 0 0" rpy="0 0 0" />
-                <geometry>
-                    <box size="${chassis_x} ${chassis_y} ${chassis_z}"/> />
-                </geometry>
-                <material name="black"/>
-            </visual>
-            <collision>
-                <origin xyz="0 0 0" rpy="0 0 0" />
-                <geometry>
-                    <box size="${chassis_x} ${chassis_y} ${chassis_z}"/> />
-                </geometry>
-            </collision>
-        </link>
-        <!-- kdl does not support a root link with an inertia, create a dummy link only contains inertia of base_link -->
-        <joint name="chassis-chassis_inertial" type="fixed">
-            <origin xyz="0 0 0" rpy="0 0 0" />
-            <parent link="chassis" />
-            <child link="chassis_inertial" />
-        </joint>
-        <link name="chassis_inertial">
-            <inertial>
-                <mass value="${chassis_m}"/>
-                <origin rpy="0 0 0" xyz="0 0 0"/>
-                <inertia ixx="${1/12*chassis_m*(chassis_y*chassis_y+chassis_z*chassis_z)}" ixy="0" ixz="0" iyy="${1/12*chassis_m*(chassis_z*chassis_z+chassis_x*chassis_x)}" iyz="0" izz="${1/12*chassis_m*(chassis_x*chassis_x+chassis_y*chassis_y)}"/>
-            </inertial>
-        </link>
-        <!-- left wheel -->
-        <joint name="$chassis-left_wheel" type="continuous">
-            <origin xyz="-${wheelbase/2} ${track/2} 0" rpy="0 0 0" />
-            <parent link="chassis"/>
-            <child link="left_wheel"/>
-            <axis xyz="0 1 0" rpy="0 0 0" />
-        </joint>
-        <link name="left_wheel">
-            <visual>
-                <origin rpy="${PI/2} 0 0" xyz="0 0 0"/>
-                <geometry>
-                    <cylinder length="${wheel_l}" radius="${wheel_r}"/>
-                </geometry>
-                <material name="orange"/>
-            </visual>
-            <collision>
-                <origin rpy="${PI/2} 0 0" xyz="0 0 0" />
-                <geometry>
-                    <cylinder length="${wheel_l}" radius="${wheel_r}"/>
-                </geometry>
-            </collision>
-            <inertial>
-                <mass value="${wheel_m}"/>
-                <origin rpy="${PI/2} 0 0" xyz="0 0 0"/>
-                <inertia ixx="${1/12*wheel_m*(3*wheel_r*wheel_r+wheel_l*wheel_l)}" ixy="0" ixz="0" iyy="${1/12*wheel_m*(3*wheel_r*wheel_r+wheel_l*wheel_l)}" iyz="0" izz="${1/2*wheel_m*wheel_r*wheel_r}"/>
-            </inertial>
-        </link>
-        <!-- right wheel -->
-        <joint name="$chassis-right_wheel" type="continuous">
-            <origin xyz="-${wheelbase/2} -${track/2} 0" rpy="0 0 0" />
-            <parent link="chassis"/>
-            <child link="right_wheel"/>
-            <axis xyz="0 1 0" rpy="0 0 0" />
-        </joint>
-        <link name="right_wheel">
-            <visual>
-                <origin rpy="${PI/2} 0 0" xyz="0 0 0"/>
-                <geometry>
-                    <cylinder length="${wheel_l}" radius="${wheel_r}"/>
-                </geometry>
-                <material name="orange"/>
-            </visual>
-            <collision>
-                <origin rpy="${PI/2} 0 0" xyz="0 0 0" />
-                <geometry>
-                    <cylinder length="${wheel_l}" radius="${wheel_r}"/>
-                </geometry>
-            </collision>
-            <inertial>
-                <mass value="${wheel_m}"/>
-                <origin rpy="${PI/2} 0 0" xyz="0 0 0"/>
-                <inertia ixx="${1/12*wheel_m*(3*wheel_r*wheel_r+wheel_l*wheel_l)}" ixy="0" ixz="0" iyy="${1/12*wheel_m*(3*wheel_r*wheel_r+wheel_l*wheel_l)}" iyz="0" izz="${1/2*wheel_m*wheel_r*wheel_r}"/>
-            </inertial>
-        </link>
-        <!-- caster ball -->
-        <joint name="joint_chassis_caster" type="fixed">
-            <origin rpy="0 0 0" xyz="${wheelbase/2} 0 -${chassis_z/2}"/>
-            <parent link="chassis"/>
-            <child link="caster"/>
-        </joint>
-        <link name="caster">
-            <visual>
-                <origin rpy="0 0 0" xyz="0 0 0"/>
-                <geometry>
-                    <sphere radius="${caster_r}"/>
-                </geometry>
-                <material name="grey"/>
-            </visual>
-            <collision>
-                <origin rpy=" 0 0 0" xyz="0 0 0"/>
-                <geometry>
-                    <sphere radius="${caster_r}"/>
-                </geometry>
-            </collision>
-            <inertial>
-                <mass value="${caster_m}"/>
-                <origin rpy="0 0 0" xyz="0 0 0"/>
-                <inertia ixx="${2/5*caster_m*caster_r*caster_r}" ixy="0" ixz="0" iyy="${2/5*caster_m*caster_r*caster_r}" iyz="0" izz="${2/5*caster_m*caster_r*caster_r}"/>
-            </inertial>
-        </link>
-        <joint name="chassis-support" type="fixed">
-            <origin rpy="0 0 0" xyz="-${wheelbase/4} 0 ${chassis_z/2+support_l/2}"/>
-            <parent link="chassis"/>
-            <child link="support"/>
-        </joint>
-        <link name="support">
-            <visual>
-                <origin rpy="0 0 0" xyz="0 0 0"/>
-                <geometry>
-                    <cylinder length="${support_l}" radius="${support_r}"/>
-                </geometry>
-                <material name="grey"/>
-            </visual>
-            <collision>
-                <origin rpy="0 0 0" xyz="0 0 0" />
-                <geometry>
-                    <cylinder length="${support_l}" radius="${support_r}"/>
-                </geometry>
-            </collision>
-            <inertial>
-                <mass value="${support_m}"/>
-                <origin rpy="0 0 0" xyz="0 0 0"/>
-                <inertia ixx="${1/12*support_m*(3*support_r*support_r+support_l*support_l)}" ixy="0" ixz="0" iyy="${1/12*support_m*(3*support_r*support_r+support_l*support_l)}" iyz="0" izz="${1/2*support_m*support_r*support_r}"/>
-            </inertial>
-        </link>
-        <joint name="support-plate" type="revolute">
-            <origin rpy="0 0 0" xyz="0 0 ${support_l/2+plate_l/2}"/>
-            <parent link="support"/>
-            <child link="plate"/>
-            <limit effort="0" lower="0" upper="0" velocity="0"/>
-            <axis rpy="0 0 0" xyz="0 0 1"/>
-        </joint>
-        <link name="plate">
-            <visual>
-                <origin rpy="0 0 0" xyz="0 0 0"/>
-                <geometry>
-                    <cylinder length="${plate_l}" radius="${plate_r}"/>
-                </geometry>
-                <material name="white"/>
-            </visual>
-            <collision>
-                <origin rpy="0 0 0" xyz="0 0 0" />
-                <geometry>
-                    <cylinder length="${plate_l}" radius="${plate_r}"/>
-                </geometry>
-            </collision>
-            <inertial>
-                <mass value="${plate_m}"/>
-                <origin rpy="0 0 0" xyz="0 0 0"/>
-                <inertia ixx="${1/12*plate_m*(3*plate_r*plate_r+plate_l*plate_l)}" ixy="0" ixz="0" iyy="${1/12*plate_m*(3*plate_r*plate_r+plate_l*plate_l)}" iyz="0" izz="${1/2*plate_m*plate_r*plate_r}"/>
-            </inertial>
-        </link>
-        <joint name="chassis-imu" type="revolute">
-            <origin rpy="0 0 0" xyz="${chassis_x/4} 0 ${chassis_z/2}"/>
-            <parent link="chassis"/>
-            <child link="imu"/>
-            <limit lower="0" upper="0" effort="0" velocity="0"/>
-            <axis xyz="0 0 1"/>
-        </joint>
-        <link name="imu"/>
-        <transmission name="left_wheel-trans" type="simpletransmission">
-            <type>transmission_interface/simpletransmission</type>
-            <actuator name="left_wheel-motor">
-                <mechanicalreduction>1</mechanicalreduction>
-            </actuator>
-            <joint name="chassis-left_wheel">
-                <hardwareinterface>hardware_interface/velocityjointinterface</hardwareinterface>
-            </joint>
-        </transmission>
-        <transmission name="right_wheel-trans" type="simpletransmission">
-            <type>transmission_interface/simpletransmission</type>
-            <actuator name="right_wheel-motor">
-                <mechanicalreduction>1</mechanicalreduction>
-            </actuator>
-            <joint name="chassis-right_wheel">
-                <hardwareinterface>hardware_interface/velocityjointinterface</hardwareinterface>
-            </joint>
-        </transmission>
-        <gazebo reference="imu">
-            <gravity>true</gravity>
-            <sensor name="imu_sensor" type="imu">
-                <always_on>true</always_on>
-                <update_rate>100</update_rate>
-                <visualize>true</visualize>
-                <topic>__default_topic__</topic>
-                <plugin filename="libgazebo_ros_imu_sensor.so" name="imu_plugin">
-                    <topicName>imu</topicName>
-                    <bodyName>imu_link</bodyName>
-                    <updateRateHZ>10.0</updateRateHZ>
-                    <gaussianNoise>0.0</gaussianNoise>
-                    <xyzOffset>0 0 0</xyzOffset>
-                    <rpyOffset>0 0 0</rpyOffset>
-                    <frameName>imu_link</frameName>
-                </plugin>
-                <pose>0 0 0 0 0 0</pose>
-            </sensor>
-        </gazebo>
-    </xacro:macro>
+<?xml version="1.0"?>
+<robot name="triwheeler" xmlns:xacro="https://www.ros.org/wiki/xacro" >
+    <!-- Included URDF Files -->
+    <xacro:include filename="$(find simbot_description)/urdf/triwheeler.urdf.xacro" />
+    <!-- Instantiate triwheeler_base_macro once (has no parameters atm) -->
+    <xacro:triwheeler_base_macro />
 </robot>

File: simbot_description/urdf/triwheeler_manipulator_rgbd.urdf.xacro (robot description, xacro)
@@ -2,5 +2,5 @@
 <robot name="triwheeler" xmlns:xacro="https://www.ros.org/wiki/xacro" >
     <!-- Included URDF Files -->
-    <xacro:include filename="$(find simbot_description)/urdf/triwheeler_base.urdf.xacro" />
+    <xacro:include filename="$(find simbot_description)/urdf/triwheeler.urdf.xacro" />
     <!-- Instantiate triwheeler_base_macro once (has no parameters atm) -->
     <xacro:triwheeler_base_macro />

File: simbot_description/urdf/triwheeler_manipulator_rgbd_laser.urdf.xacro (robot description, xacro)
@@ -2,5 +2,5 @@
 <robot name="triwheeler" xmlns:xacro="https://www.ros.org/wiki/xacro" >
     <!-- Included URDF Files -->
-    <xacro:include filename="$(find simbot_description)/urdf/triwheeler_base.urdf.xacro" />
+    <xacro:include filename="$(find simbot_description)/urdf/triwheeler.urdf.xacro" />
     <!-- Instantiate triwheeler_base_macro once (has no parameters atm) -->
     <xacro:triwheeler_base_macro />

File: simbot_description/urdf/triwheeler_rgbd.urdf.xacro (robot description, xacro)
@@ -2,5 +2,5 @@
 <robot name="triwheeler" xmlns:xacro="https://www.ros.org/wiki/xacro" >
     <!-- Included URDF Files -->
-    <xacro:include filename="$(find simbot_description)/urdf/triwheeler_base.urdf.xacro" />
+    <xacro:include filename="$(find simbot_description)/urdf/triwheeler.urdf.xacro" />
     <!-- Instantiate triwheeler_base_macro once (has no parameters atm) -->
     <xacro:triwheeler_base_macro />

Commit message: add gazebo markups

File: simbot_description/urdf/triwheeler.urdf.xacro (robot description, xacro)
@@ -48,4 +48,9 @@
             </collision>
         </link>
+        <gazebo reference="chassis">
+            <mu1>0.2</mu1>
+            <mu2>0.2</mu2>
+            <material>Gazebo/Black</material>
+        </gazebo>
         <!-- kdl does not support a root link with an inertia, create a dummy link only contains inertia of base_link -->
         <joint name="chassis-chassis_inertial" type="fixed">
@@ -88,4 +93,9 @@
             </inertial>
         </link>
+        <gazebo reference="left_wheel">
+            <mu1>0.99</mu1>
+            <mu2>0.99</mu2>
+            <material>Gazebo/Wood</material>
+        </gazebo>
         <!-- right wheel -->
         <joint name="$chassis-right_wheel" type="continuous">
@@ -115,4 +125,9 @@
             </inertial>
         </link>
+        <gazebo reference="right_wheel">
+            <mu1>0.99</mu1>
+            <mu2>0.99</mu2>
+            <material>Gazebo/Wood</material>
+        </gazebo>
         <!-- caster ball -->
         <joint name="joint_chassis_caster" type="fixed">
@@ -141,4 +156,9 @@
             </inertial>
         </link>
+        <gazebo reference="caster">
+            <mu1>0.0</mu1>
+            <mu2>0.0</mu2>
+            <material>Gazebo/Grey</material>
+        </gazebo>
         <joint name="chassis-support" type="fixed">
             <origin rpy="0 0 0" xyz="-${wheelbase/4} 0 ${chassis_z/2+support_l/2}"/>
@@ -166,4 +186,9 @@
             </inertial>
         </link>
+        <gazebo reference="support">
+            <mu1>0.2</mu1>
+            <mu2>0.2</mu2>
+            <material>Gazebo/Grey</material>
+        </gazebo>
         <joint name="support-plate" type="revolute">
             <origin rpy="0 0 0" xyz="0 0 ${support_l/2+plate_l/2}"/>
@@ -193,4 +218,9 @@
             </inertial>
         </link>
+        <gazebo reference="plate">
+            <mu1>0.77</mu1>
+            <mu2>0.77</mu2>
+            <material>Gazebo/CoM</material>
+        </gazebo>
         <joint name="chassis-imu" type="revolute">
             <origin rpy="0 0 0" xyz="${chassis_x/4} 0 ${chassis_z/2}"/>

File: simbot_description/urdf/triwheeler_manipulator_rgbd_laser.urdf.xacro (robot description, xacro)
@@ -5,4 +5,10 @@
     <!-- Instantiate triwheeler_base_macro once (has no parameters atm) -->
     <xacro:triwheeler_base_macro />
+    <gazebo>
+        <plugin name="gazebo_ros_control" filename="libgazebo_ros_control.so">
+            <robotNamespace>/triwheeler</robotNamespace>
+            <robotSimType>gazebo_ros_control/DefaultRobotHWSim</robotSimType>
+        </plugin>
+    </gazebo>
     <!-- manipulator -->
     <xacro:include filename="$(find simbot_description)/urdf/manipulator.urdf.xacro" />

Commit message: add control package: HWinterface not working

File: simbot_description/urdf/triwheeler.urdf.xacro (robot description, xacro)
@@ -67,5 +67,5 @@
         </link>
         <!-- left wheel -->
-        <joint name="$chassis-left_wheel" type="continuous">
+        <joint name="chassis-left_wheel" type="continuous">
             <origin xyz="-${wheelbase/2} ${track/2} 0" rpy="0 0 0" />
             <parent link="chassis"/>
@@ -237,5 +237,5 @@
             </actuator>
             <joint name="chassis-left_wheel">
-                <hardwareinterface>hardware_interface/velocityjointinterface</hardwareinterface>
+                <hardwareinterface>hardware_interface/VelocityJointInterface</hardwareinterface>
             </joint>
         </transmission>
@@ -246,7 +246,13 @@
             </actuator>
             <joint name="chassis-right_wheel">
-                <hardwareinterface>hardware_interface/velocityjointinterface</hardwareinterface>
+                <hardwareinterface>hardware_interface/VelocityJointInterface</hardwareinterface>
             </joint>
         </transmission>
+        <gazebo>
+            <plugin name="gazebo_ros_control" filename="libgazebo_ros_control.so">
+                <robotNamespace>/triwheeler</robotNamespace>
+                <robotSimType>gazebo_ros_control/DefaultRobotHWSim</robotSimType>
+            </plugin>
+        </gazebo>
         <gazebo reference="imu">
             <gravity>true</gravity>

File: simbot_description/urdf/triwheeler_manipulator_rgbd_laser.urdf.xacro (robot description, xacro)
@@ -5,10 +5,4 @@
     <!-- Instantiate triwheeler_base_macro once (has no parameters atm) -->
     <xacro:triwheeler_base_macro />
-    <gazebo>
-        <plugin name="gazebo_ros_control" filename="libgazebo_ros_control.so">
-            <robotNamespace>/triwheeler</robotNamespace>
-            <robotSimType>gazebo_ros_control/DefaultRobotHWSim</robotSimType>
-        </plugin>
-    </gazebo>
     <!-- manipulator -->
     <xacro:include filename="$(find simbot_description)/urdf/manipulator.urdf.xacro" />
